Commit message: collada model file for erratic robot, add missing dependency on pr2_simulator stack which contains controller manager plugin

File: erratic_description/urdf/erratic_base.xacro (robot description, xacro)
@@ -65,5 +65,5 @@
                 <origin xyz="0.0 0.0 0.0" rpy="0 0 0" />
                 <geometry>
-                    <box size="${base_size_x} ${base_size_y} ${base_size_z}" />
+                    <mesh filename="package://erratic_description/meshes/collada/base_link.dae"/>
                 </geometry>
                 <material name="Blue" />
@@ -72,5 +72,5 @@
                 <origin xyz="0.0 0.0 0.0" rpy="0 0 0" />
                 <geometry>
-                    <box size="${base_size_x} ${base_size_y} ${base_size_z}" />
+                    <mesh filename="package://erratic_description/meshes/collada/base_link.dae"/>
                 </geometry>
             </collision>
@@ -92,5 +92,5 @@
                 <origin xyz="0.0 0.0 0.0" rpy="0 0 0" />
                 <geometry>
-                    <mesh filename="package://erratic_description/meshes/erratic_top.stl"/>
+                    <mesh filename="package://erratic_description/meshes/collada/erratic_top.dae"/>
                 </geometry>
                 <material name="Blue" />
@@ -99,38 +99,11 @@
                 <origin xyz="0.0 0.0 0.0" rpy="0 0 0" />
                 <geometry>
-                    <mesh filename="package://erratic_description/meshes/erratic_top.stl"/>
-                </geometry>
-            </collision>
-        </link>
-        <joint name="base_caster_box_joint" type="fixed">
-            <origin xyz="-${base_size_x/2 + caster_support_x/2} 0 ${base_size_z/2 - caster_support_z/2}" rpy="0 0 0" />
+                    <mesh filename="package://erratic_description/meshes/collada/erratic_top.dae"/>
+                </geometry>
+            </collision>
+        </link>
+        <joint name="base_caster_support_joint" type="continuous">
+            <origin xyz="${-0.194 + 0.015} 0 ${-0.032 - 0.0315}" rpy="0 0 0" />
             <parent link="base_link" />
-            <child link="base_caster_box_link"/>
-        </joint>
-        <link name="base_caster_box_link">
-            <inertial>
-                <mass value="0.1"/>
-                <origin xyz="0 0 0" />
-                <inertia ixx="0.01" ixy="0.0" ixz="0.0"
-                         iyy="0.01" iyz="0.0"
-                         izz="0.01" />
-            </inertial>
-            <visual>
-                <origin xyz="0.0 0.0 0.0" rpy="0 0 0" />
-                <geometry>
-                    <box size="${caster_support_x} 0.02 ${caster_support_z}" />
-                </geometry>
-                <material name="Blue" />
-            </visual>
-            <collision>
-                <origin xyz="0.0 0.0 0.0" rpy="0 0 0" />
-                <geometry>
-                    <box size="${caster_support_x} 0.02 ${caster_support_z}" />
-                </geometry>
-            </collision>
-        </link>
-        <joint name="base_caster_support_joint" type="continuous">
-            <origin xyz="${-caster_support_x/2 + 0.015} 0 ${-caster_support_z/2 - 0.0315}" rpy="0 0 0" />
-            <parent link="base_caster_box_link" />
             <child link="base_caster_support_link"/>
             <axis xyz="0 0 1" />
@@ -155,11 +128,11 @@
                 <origin xyz="0.0 0.0 0.0" rpy="0 0 0" />
                 <geometry>
-                    <box size="0.03 0.02 0.063" />
-                </geometry>
-            </visual>
-            <collision>
-                <origin xyz="0.0 0.0 0.0" rpy="0 0 0" />
-                <geometry>
-                    <box size="0.03 0.02 0.063" />
+                    <mesh filename="package://erratic_description/meshes/collada/caster_support.dae"/>
+                </geometry>
+            </visual>
+            <collision>
+                <origin xyz="0.0 0.0 0.0" rpy="0 0 0" />
+                <geometry>
+                    <mesh filename="package://erratic_description/meshes/collada/caster_support.dae"/>
                 </geometry>
             </collision>
@@ -190,5 +163,5 @@
                 <origin xyz="0 0 0" rpy="${M_PI/2} 0 0" />
                 <geometry>
-                    <cylinder radius="0.035" length="0.01" />
+                    <mesh filename="package://erratic_description/meshes/collada/caster_wheel.dae"/>
                 </geometry>
                 <material name="Black"/>
@@ -197,5 +170,5 @@
             <origin xyz="0 0 0" rpy="${M_PI/2} 0 0" />
             <geometry>
-                <cylinder radius="0.035" length="0.01" />
+                <mesh filename="package://erratic_description/meshes/collada/caster_wheel.dae"/>
             </geometry>
             </collision>

File: erratic_description/urdf/erratic_wheel.xacro (robot description, xacro)
@@ -8,37 +8,11 @@
     <property name="wheel_offset_z" value="${-base_size_z/2 + 0.0236}" />
     <macro name="erratic_wheel" params="suffix parent reflect">
-        <joint name="${parent}_${suffix}_motor_joint" type="fixed">
-            <origin xyz="0.075 ${reflect*base_size_y/2} ${wheel_offset_z}" rpy="0 0 0" />
-            <parent link="${parent}" />
-            <child link="${parent}_${suffix}_motor_link" />
-        </joint>
-        <link name="${parent}_${suffix}_motor_link">
-            <inertial>
-                <mass value="0.1" />
-                <origin xyz=" 0 ${reflect*0.0125} 0 " />
-                <inertia  ixx="0.012411765597" ixy="0.0" ixz="0.0"
-                          iyy="0.015218160428" iyz="0.0"
-                          izz="0.011763977943" />
-            </inertial>
-            <visual>
-                <origin xyz="0 ${reflect*0.0125} 0" rpy="${M_PI/2} 0 0" />
-                <geometry>
-                    <cylinder radius="0.0127" length="0.025" />
-                </geometry>
-            </visual>
-            <collision>
-                <origin xyz="0 ${reflect*0.0125} 0" rpy="${M_PI/2} 0 0" />
-                <geometry>
-                    <cylinder radius="0.0127" length="0.025" />
-                </geometry>
-            </collision>
-        </link>
         <joint name="${parent}_${suffix}_wheel_joint" type="continuous">
-            <origin xyz="0 ${reflect*0.025} 0" rpy="0 0 0" />
+            <origin xyz="0.075 ${reflect*0.165} -0.0539" rpy="0 0 0" />
             <axis xyz="0 1 0" />
             <anchor xyz="0 0 0" />
             <limit effort="100" velocity="100" />
             <joint_properties damping="0.0" friction="0.0" />
-            <parent link="${parent}_${suffix}_motor_link" />
+            <parent link="${parent}" />
             <child link="${parent}_${suffix}_wheel_link" />
         </joint>
@@ -54,5 +28,5 @@
                 <origin xyz="0 0 0" rpy="0 0 ${M_PI/2}" />
                 <geometry>
-                    <mesh filename="package://erratic_description/meshes/erratic_wheel.stl"/>
+                    <mesh filename="package://erratic_description/meshes/collada/erratic_wheel.dae"/>
                 </geometry>
                 <material name="Black" />
@@ -61,5 +35,5 @@
                 <origin xyz="0 0 0" rpy="0 0 ${M_PI/2}" />
                 <geometry>
-                    <mesh filename="package://erratic_description/meshes/erratic_wheel.stl"/>
+                    <mesh filename="package://erratic_description/meshes/collada/erratic_wheel.dae"/>
                 </geometry>
             </collision>

Commit message: dae to stl

File: erratic_description/urdf/erratic_base.xacro (robot description, xacro)
@@ -65,5 +65,5 @@
                 <origin xyz="0.0 0.0 0.0" rpy="0 0 0" />
                 <geometry>
-                    <mesh filename="package://erratic_description/meshes/collada/base_link.dae"/>
+                    <mesh filename="package://erratic_description/meshes/base_link.stl"/>
                 </geometry>
                 <material name="Blue" />
@@ -72,5 +72,5 @@
                 <origin xyz="0.0 0.0 0.0" rpy="0 0 0" />
                 <geometry>
-                    <mesh filename="package://erratic_description/meshes/collada/base_link.dae"/>
+                    <mesh filename="package://erratic_description/meshes/base_link.stl"/>
                 </geometry>
             </collision>
@@ -92,5 +92,5 @@
                 <origin xyz="0.0 0.0 0.0" rpy="0 0 0" />
                 <geometry>
-                    <mesh filename="package://erratic_description/meshes/collada/erratic_top.dae"/>
+                    <mesh filename="package://erratic_description/meshes/erratic_top.stl"/>
                 </geometry>
                 <material name="Blue" />
@@ -99,5 +99,5 @@
                 <origin xyz="0.0 0.0 0.0" rpy="0 0 0" />
                 <geometry>
-                    <mesh filename="package://erratic_description/meshes/collada/erratic_top.dae"/>
+                    <mesh filename="package://erratic_description/meshes/erratic_top.stl"/>
                 </geometry>
             </collision>
@@ -128,11 +128,11 @@
                 <origin xyz="0.0 0.0 0.0" rpy="0 0 0" />
                 <geometry>
-                    <mesh filename="package://erratic_description/meshes/collada/caster_support.dae"/>
-                </geometry>
-            </visual>
-            <collision>
-                <origin xyz="0.0 0.0 0.0" rpy="0 0 0" />
-                <geometry>
-                    <mesh filename="package://erratic_description/meshes/collada/caster_support.dae"/>
+                    <mesh filename="package://erratic_description/meshes/caster_support.stl"/>
+                </geometry>
+            </visual>
+            <collision>
+                <origin xyz="0.0 0.0 0.0" rpy="0 0 0" />
+                <geometry>
+                    <mesh filename="package://erratic_description/meshes/caster_support.stl"/>
                 </geometry>
             </collision>
@@ -163,5 +163,5 @@
                 <origin xyz="0 0 0" rpy="${M_PI/2} 0 0" />
                 <geometry>
-                    <mesh filename="package://erratic_description/meshes/collada/caster_wheel.dae"/>
+                    <mesh filename="package://erratic_description/meshes/caster_wheel.stl"/>
                 </geometry>
                 <material name="Black"/>
@@ -170,5 +170,5 @@
             <origin xyz="0 0 0" rpy="${M_PI/2} 0 0" />
             <geometry>
-                <mesh filename="package://erratic_description/meshes/collada/caster_wheel.dae"/>
+                <mesh filename="package://erratic_description/meshes/caster_wheel.stl"/>
             </geometry>
             </collision>

File: erratic_description/urdf/erratic_wheel.xacro (robot description, xacro)
@@ -28,5 +28,5 @@
                 <origin xyz="0 0 0" rpy="0 0 ${M_PI/2}" />
                 <geometry>
-                    <mesh filename="package://erratic_description/meshes/collada/erratic_wheel.dae"/>
+                    <mesh filename="package://erratic_description/meshes/erratic_wheel.stl"/>
                 </geometry>
                 <material name="Black" />
@@ -35,5 +35,5 @@
                 <origin xyz="0 0 0" rpy="0 0 ${M_PI/2}" />
                 <geometry>
-                    <mesh filename="package://erratic_description/meshes/collada/erratic_wheel.dae"/>
+                    <mesh filename="package://erratic_description/meshes/erratic_wheel.stl"/>
                 </geometry>
             </collision>

Commit message: Erratic robot demos should run on diamondback

File: erratic_description/urdf/erratic_base.xacro (robot description, xacro)
@@ -72,5 +72,5 @@
                 <origin xyz="0.0 0.0 0.0" rpy="0 0 0" />
                 <geometry>
-                    <mesh filename="package://erratic_description/meshes/base_link.stl"/>
+                    <mesh filename="package://erratic_description/meshes/collada/base_link.dae"/>
                 </geometry>
             </collision>
@@ -99,5 +99,5 @@
                 <origin xyz="0.0 0.0 0.0" rpy="0 0 0" />
                 <geometry>
-                    <mesh filename="package://erratic_description/meshes/erratic_top.stl"/>
+                    <mesh filename="package://erratic_description/meshes/collada/erratic_top.dae"/>
                 </geometry>
             </collision>
@@ -134,5 +134,5 @@
                 <origin xyz="0.0 0.0 0.0" rpy="0 0 0" />
                 <geometry>
-                    <mesh filename="package://erratic_description/meshes/caster_support.stl"/>
+                    <mesh filename="package://erratic_description/meshes/collada/caster_support.dae"/>
                 </geometry>
             </collision>
@@ -170,5 +170,5 @@
             <origin xyz="0 0 0" rpy="${M_PI/2} 0 0" />
             <geometry>
-                <mesh filename="package://erratic_description/meshes/caster_wheel.stl"/>
+                <mesh filename="package://erratic_description/meshes/collada/caster_wheel.dae"/>
             </geometry>
             </collision>

File: erratic_description/urdf/erratic_wheel.xacro (robot description, xacro)
@@ -35,5 +35,5 @@
                 <origin xyz="0 0 0" rpy="0 0 ${M_PI/2}" />
                 <geometry>
-                    <mesh filename="package://erratic_description/meshes/erratic_wheel.stl"/>
+                    <mesh filename="package://erratic_description/meshes/collada/erratic_wheel.dae"/>
                 </geometry>
             </collision>
