Commit message: update erratic meshes, more size-shape accurate

File: erratic_description/urdf/erratic_base.xacro (robot description, xacro)
@@ -8,17 +8,7 @@
     <include filename="$(find erratic_description)/urdf/erratic_computer.xacro" />
     <include filename="$(find erratic_description)/urdf/erratic_wheel.xacro" />
-    <!-- Properties (Constants) -->
-    <property name="M_PI" value="3.14159"/>
-    <property name="base_size_x" value="0.217" />
-    <property name="base_size_y" value="0.280" />
-    <property name="base_size_z" value="0.155" />
-    <property name="top_size_x" value="0.3937" />
-    <property name="top_size_y" value="0.3556" />
-    <property name="top_size_z" value="0.0020" />
-    <property name="wheel_radius" value="0.0746" />
-    <property name="wheel_length" value="0.02" />
-    <property name="caster_wheel_offset_y" value="0.17" />
-    <property name="caster_support_x" value="0.086" />
-    <property name="caster_support_z" value="0.1095" />
+    <property name="base_link_to_top" value="0.0795" />
+    <property name="base_link_to_front" value="0.2025" />
+    <property name="base_link_to_back" value="0.1975" />
     <macro name="erratic">
         <!-- base_footprint is a fictitious link(frame) that is on the ground right below base_link origin,
@@ -40,5 +30,5 @@
             </visual>
             <collision>
-                <origin xyz="0 0 ${base_size_z/2 + 0.051}" rpy="0 0 0" />
+                <origin xyz="0 0 0.128" rpy="0 0 0" />
                 <geometry>
                   <box size="0.001 0.001 0.001" />
@@ -47,7 +37,5 @@
         </link>
         <joint name="base_footprint_joint" type="fixed">
-            <!-- NB: While you would think this would make it go up, it is oddly reversed.
-                 This moves the joint to 0,0,0 where we want it for rviz, etc. -->
-            <origin xyz="0 0 ${base_size_z/2 + 0.051}" rpy="0 0 0" />
+            <origin xyz="0 0 0.128" rpy="0 0 0" />
             <parent link="base_footprint"/>
             <child link="base_link" />
@@ -57,5 +45,5 @@
             <inertial>
                 <mass value="20" />
-                <origin xyz="${-base_size_x/2} 0 ${-base_size_z/2}" />
+                <origin xyz="0 0 0" />
                 <inertia ixx="1.0" ixy="0.0" ixz="0.0"
                          iyy="1.0" iyz="0.0"
@@ -63,46 +51,19 @@
             </inertial>
             <visual>
-                <origin xyz="0.0 0.0 0.0" rpy="0 0 0" />
-                <geometry>
-                    <mesh filename="package://erratic_description/meshes/base_link.stl"/>
+                <origin xyz="0 0 0" rpy="0 0 0" />
+                <geometry>
+                    <mesh filename="package://erratic_description/meshes/collada/erratic_base_link.dae"/>
                 </geometry>
                 <material name="Blue" />
             </visual>
             <collision>
-                <origin xyz="0.0 0.0 0.0" rpy="0 0 0" />
-                <geometry>
-                    <mesh filename="package://erratic_description/meshes/collada/base_link.dae"/>
-                </geometry>
-            </collision>
-        </link>
-        <joint name="base_top_joint" type="fixed" >
-            <origin xyz="0 0 ${base_size_z/2 + top_size_z/2}" rpy="0 0 0" />   <!-- 0.051 -->
-            <parent link="base_link" />
-            <child link="base_top_link"/>
-        </joint>
-        <link name="base_top_link">
-            <inertial>
-                <mass value="1.0"/>
-                <origin xyz="-0.00125736 0.0 -0.0032368" />
-                <inertia ixx="0.00995424" ixy="0.0" ixz="0.00000413"
-                         iyy="0.01191941" iyz="0.0" izx="0.00000413"
-                         izz="0.02181097" />
-            </inertial>
-            <visual>
-                <origin xyz="0.0 0.0 0.0" rpy="0 0 0" />
-                <geometry>
-                    <mesh filename="package://erratic_description/meshes/erratic_top.stl"/>
-                </geometry>
-                <material name="Blue" />
-            </visual>
-            <collision>
-                <origin xyz="0.0 0.0 0.0" rpy="0 0 0" />
-                <geometry>
-                    <mesh filename="package://erratic_description/meshes/collada/erratic_top.dae"/>
+                <origin xyz="0 0 0" rpy="0 0 0" />
+                <geometry>
+                    <mesh filename="package://erratic_description/meshes/collada/erratic_base_link.dae"/>
                 </geometry>
             </collision>
         </link>
         <joint name="base_caster_support_joint" type="continuous">
-            <origin xyz="${-0.194 + 0.015} 0 ${-0.032 - 0.0315}" rpy="0 0 0" />
+            <origin xyz="-0.188 0 -0.043" rpy="0 0 0" />
             <parent link="base_link" />
             <child link="base_caster_support_link"/>
@@ -126,18 +87,18 @@
             </inertial>
             <visual>
-                <origin xyz="0.0 0.0 0.0" rpy="0 0 0" />
-                <geometry>
-                    <mesh filename="package://erratic_description/meshes/caster_support.stl"/>
-                </geometry>
-            </visual>
-            <collision>
-                <origin xyz="0.0 0.0 0.0" rpy="0 0 0" />
-                <geometry>
-                    <mesh filename="package://erratic_description/meshes/collada/caster_support.dae"/>
+                <origin xyz="0 0 0" rpy="0 0 0" />
+                <geometry>
+                    <mesh filename="package://erratic_description/meshes/collada/erratic_caster_support_link.dae"/>
+                </geometry>
+            </visual>
+            <collision>
+                <origin xyz="0 0 0" rpy="0 0 0" />
+                <geometry>
+                    <mesh filename="package://erratic_description/meshes/collada/erratic_caster_support_link.dae"/>
                 </geometry>
             </collision>
         </link>
         <joint name="caster_wheel_joint" type="continuous">
-            <origin xyz="-0.015 0 -0.03" rpy="0 0 0" />
+            <origin xyz="-0.025 0 -0.0469" rpy="0 0 0" />
             <parent link="base_caster_support_link" />
             <child link="caster_wheel_link" />
@@ -155,5 +116,5 @@
             <inertial>
                 <mass value="0.1" />
-                <origin xyz="0.0 0.0 0.0" rpy="0 0 0" />
+                <origin xyz="0 0 0" rpy="0 0 0" />
                 <inertia  ixx="0.012411765597" ixy="-0.000711733678" ixz="0.00050272983"
                           iyy="0.015218160428" iyz="-0.000004273467"
@@ -161,15 +122,15 @@
             </inertial>
             <visual>
-                <origin xyz="0 0 0" rpy="${M_PI/2} 0 0" />
-                <geometry>
-                    <mesh filename="package://erratic_description/meshes/caster_wheel.stl"/>
+                <origin xyz="0 0 0" rpy="0 0 0" />
+                <geometry>
+                    <mesh filename="package://erratic_description/meshes/collada/erratic_caster_wheel_link.dae"/>
                 </geometry>
                 <material name="Black"/>
             </visual>
             <collision>
-            <origin xyz="0 0 0" rpy="${M_PI/2} 0 0" />
-            <geometry>
-                <mesh filename="package://erratic_description/meshes/collada/caster_wheel.dae"/>
-            </geometry>
+                <origin xyz="0 0 0" rpy="0 0 0" />
+                <geometry>
+                    <mesh filename="package://erratic_description/meshes/collada/erratic_caster_wheel_link.dae"/>
+                </geometry>
             </collision>
         </link>
@@ -181,7 +142,13 @@
         </gazebo>
         <!-- MACRO INSTANTIATION -->
-        <erratic_computer parent="base_top_link"/>
-        <erratic_wheel suffix="left" parent="base_link" reflect="1"/>
-        <erratic_wheel suffix="right" parent="base_link" reflect="-1"/>
+        <erratic_computer parent="base_link">
+            <origin xyz="${-base_link_to_back + computer_size_x/2 + 0.02} 0 ${base_link_to_top}" rpy="0 0 0" />
+        </erratic_computer>
+        <erratic_wheel suffix="left" parent="base_link">
+            <origin xyz="0.075 0.16525 -0.053" rpy="0 0 0" />
+        </erratic_wheel>
+        <erratic_wheel suffix="right" parent="base_link">
+            <origin xyz="0.075 -0.16525 -0.053" rpy="0 0 0" />
+        </erratic_wheel>
         <!-- CONTROLLERS -->
         <gazebo>
@@ -192,6 +159,6 @@
                 <leftJoint>base_link_right_wheel_joint</leftJoint>
                 <rightJoint>base_link_left_wheel_joint</rightJoint>
-                <wheelSeparation>${caster_wheel_offset_y*2}</wheelSeparation>
-                <wheelDiameter>${wheel_radius*2}</wheelDiameter>
+                <wheelSeparation>0.3305</wheelSeparation>
+                <wheelDiameter>0.15</wheelDiameter>
                 <torque>5</torque>
                 <interface:position name="position_iface_0"/>

File: erratic_description/urdf/erratic_computer.xacro (robot description, xacro)
@@ -7,7 +7,7 @@
     <property name="computer_size_y" value="0.175" />
     <property name="computer_size_z" value="0.056" />
-    <macro name="erratic_computer" params="parent">
+    <macro name="erratic_computer" params="parent *origin">
         <joint name="computer_mount_joint" type="fixed">
-            <origin xyz="-${top_size_x/2 - 0.0254 - computer_size_y/2} ${top_size_y/2 - 0.1 - computer_size_y/2} ${top_size_z/2}" />
+            <insert_block name="origin" />
             <parent link="${parent}" />
             <child link="computer_link" />

File: erratic_description/urdf/erratic_laser.urdf.xacro (robot description, xacro)
@@ -9,6 +9,6 @@
     <erratic />
     <!-- BASE LASER ATTACHMENT -->
-    <erratic_hokuyo_laser parent="base_top_link">
-        <origin xyz="${top_size_x/2 - 0.01 - 0.04} 0 ${top_size_z/2}" rpy="0 0 0" />
+    <erratic_hokuyo_laser parent="base_link">
+        <origin xyz="${base_link_to_front - 0.01 - 0.04} 0 ${base_link_to_top}" rpy="0 0 0" />
     </erratic_hokuyo_laser>
 </robot>

File: erratic_description/urdf/erratic_wheel.xacro (robot description, xacro)
@@ -4,10 +4,7 @@
     xmlns:controller="http://playerstage.sourceforge.net/gazebo/xmlschema/#controller"
     xmlns:interface="http://playerstage.sourceforge.net/gazebo/xmlschema/#interface">
-    <!-- Properties (Constants) -->
-    <property name="M_PI" value="3.14159"/>
-    <property name="wheel_offset_z" value="${-base_size_z/2 + 0.0236}" />
-    <macro name="erratic_wheel" params="suffix parent reflect">
+    <macro name="erratic_wheel" params="suffix parent *origin">
         <joint name="${parent}_${suffix}_wheel_joint" type="continuous">
-            <origin xyz="0.075 ${reflect*0.165} -0.0539" rpy="0 0 0" />
+            <insert_block name="origin" />
             <axis xyz="0 1 0" />
             <anchor xyz="0 0 0" />
@@ -26,14 +23,14 @@
             </inertial>
             <visual>
-                <origin xyz="0 0 0" rpy="0 0 ${M_PI/2}" />
+                <origin xyz="0 0 0" rpy="0 0 0" />
                 <geometry>
-                    <mesh filename="package://erratic_description/meshes/erratic_wheel.stl"/>
+                    <mesh filename="package://erratic_description/meshes/collada/erratic_front_wheel_link.dae"/>
                 </geometry>
                 <material name="Black" />
             </visual>
             <collision>
-                <origin xyz="0 0 0" rpy="0 0 ${M_PI/2}" />
+                <origin xyz="0 0 0" rpy="0 0 0" />
                 <geometry>
-                    <mesh filename="package://erratic_description/meshes/collada/erratic_wheel.dae"/>
+                    <mesh filename="package://erratic_description/meshes/collada/erratic_front_wheel_link.dae"/>
                 </geometry>
             </collision>

Commit message: add example launch files for two erratics in the same world

File: erratic_description/urdf/erratic_base.xacro (robot description, xacro)
@@ -37,5 +37,5 @@
         </link>
         <joint name="base_footprint_joint" type="fixed">
-            <origin xyz="0 0 0.128" rpy="0 0 0" />
+            <origin xyz="0.063 0 0.128" rpy="0 0 0" />
             <parent link="base_footprint"/>
             <child link="base_link" />
@@ -163,5 +163,4 @@
                 <torque>5</torque>
                 <interface:position name="position_iface_0"/>
-                <robotNamespace>/</robotNamespace>
                 <topicName>cmd_vel</topicName>
             </controller:diffdrive_plugin>
